File: hardware/esr-meter.kicad_sch (KiCad schematic)
At the start: 101 parts, among them J1 USB_B_Micro, J2 JST-XH, J3 Pin Header Male, J4 Binding Post, Q1 DTC114E, Q2 IRLML6402, Q3 DTC114E, Q4 DTC114E, Q5 MMBFJ113, Q6 DTC114E, Q7 DTC114E, Q8 DTC114E, Q9 DTC114E, SW1 SW_Push, U1 MCP73831, U2 TPS60403, U3 TLV431, U4 OPA1678, U5 OPA1678, U6 ATmega88PA-AU, U7 QDSP-6064, U8 OPA1678

Commit message: Split A2 circuit into A4 pages
Parts:
- removed C1, C6: 4.7u, Capacitor_SMD:C_1206_3216Metric, symbol Device:C
- removed C10, C15, C7, C9: 10n, Capacitor_SMD:C_0603_1608Metric, symbol Device:C
- removed C11: DNP, Capacitor_SMD:C_0603_1608Metric, symbol Device:C
- removed C12, C13, C14: 1n, Capacitor_SMD:C_0603_1608Metric, symbol Device:C
- removed C16, C17, C18, C19, C20, C21, C22, C23, C24, C3, C8: 100n, Capacitor_SMD:C_0603_1608Metric, symbol Device:C
- removed C2, C4, C5: 1u, Capacitor_SMD:C_1206_3216Metric, symbol Device:C
- removed D1: SMAJ5.0A, Diode_SMD:D_SMA, symbol Device:D_Zener
- removed D10, D11: SM4007, Diode_SMD:D_MELF, symbol Diode:SM4007
- removed D2: RED, LED_SMD:LED_1206_3216Metric, symbol Device:LED
- removed D3: GREEN, LED_SMD:LED_1206_3216Metric, symbol Device:LED
- removed D4, D5, D6, D7, D9: BAS316, Diode_SMD:D_SOD-323, symbol Diode:BAS316
- removed D8: BAT54J, Diode_SMD:D_SOD-323F, symbol Diode:BAT54J
- removed J1: USB_B_Micro, Connector_USB:USB_Micro-B_Molex-105017-0001, symbol Connector:USB_B_Micro
- removed J2: JST-XH, Connector_JST:JST_XH_S2B-XH-A-1_1x02_P2.50mm_Horizontal, symbol Connector_Generic:Conn_01x02
- removed J3: Pin Header Male, Connector_PinHeader_2.54mm:PinHeader_2x03_P2.54mm_Vertical, symbol Connector_Generic:Conn_02x03_Odd_Even
- removed J4: Binding Post, esr-meter:BindingPost, symbol Connector_Generic:Conn_01x02
- removed Q1, Q3, Q4, Q6, Q7, Q8, Q9: DTC114E, Package_TO_SOT_SMD:SOT-23, symbol Device:Q_NPN_BEC_BRT
- removed Q2: IRLML6402, Package_TO_SOT_SMD:SOT-23, symbol Transistor_FET:IRLML6402
- removed Q5: MMBFJ113, Package_TO_SOT_SMD:SOT-23, symbol Transistor_FET:MMBFJ113
- removed R1, R22, R6: 33k, Resistor_SMD:R_0603_1608Metric, symbol Device:R
- removed R10, R18, R5, R8, R9: 10k, Resistor_SMD:R_0603_1608Metric, symbol Device:R
- removed R11, R35, R36, R38, R39, R41, R42, R43, R44: 10, Resistor_SMD:R_0603_1608Metric, symbol Device:R
- removed R12, R13: 100k, Resistor_SMD:R_0603_1608Metric, symbol Device:R
- removed R14, R15, R19, R26, R37: 1k, Resistor_SMD:R_0603_1608Metric, symbol Device:R
- removed R16: DNP, Resistor_SMD:R_0603_1608Metric, symbol Device:R
- removed R17, R23: 1.58k, Resistor_SMD:R_0603_1608Metric, symbol Device:R
- removed R2: 3.3k, Resistor_SMD:R_0603_1608Metric, symbol Device:R
- removed R20: 3.3M, Resistor_SMD:R_0603_1608Metric, symbol Device:R
- removed R21: 2.2k, Resistor_SMD:R_0603_1608Metric, symbol Device:R
- removed R24: 499, Resistor_SMD:R_0805_2012Metric, symbol Device:R
- removed R25: 10, Resistor_SMD:R_0805_2012Metric, symbol Device:R
- removed R27, R28, R29, R30, R31, R32, R33, R34: 2.4k, Resistor_SMD:R_0603_1608Metric, symbol Device:R
- removed R3, R4: 3k, Resistor_SMD:R_0603_1608Metric, symbol Device:R
- removed R40: 45.3k, Resistor_SMD:R_0603_1608Metric, symbol Device:R
- removed R7: 31.6k, Resistor_SMD:R_0603_1608Metric, symbol Device:R
- removed SW1: SW_Push, Button_Switch_THT:SW_PUSH-12mm_Wuerth-430476085716, symbol Switch:SW_Push
- removed U1: MCP73831, Package_TO_SOT_SMD:SOT-23-5, symbol Battery_Management:MCP73831-2-OT
- removed U2: TPS60403, Package_TO_SOT_SMD:SOT-23-5, symbol esr-meter:TPS6040x
- removed U3: TLV431, Package_TO_SOT_SMD:SOT-23, symbol Reference_Voltage:TL431DBZ
- removed U4, U5, U8: OPA1678, Package_SO:SO-8_3.9x4.9mm_P1.27mm, symbol Amplifier_Operational:OPA1678
- removed U6: ATmega88PA-AU, Package_QFP:TQFP-32_7x7mm_P0.8mm, symbol MCU_Microchip_ATmega:ATmega88PA-A
- removed U7: QDSP-6064, Package_DIP:DIP-12_W7.62mm, symbol esr-meter:QDSP-6064
Connections:
- no-connect marks 9 -> 0
Other:
- added sheet Analog (analog.kicad_sch)
- added sheet Digital (digital.kicad_sch)
- added sheet Power (power.kicad_sch)
- note removed: "3.7V LiPo Battery"
- note removed: "50 mVpp 100 kHz"
- note removed: "AVR ISP"
- note removed: "Amplifier"
- note removed: "Capacitor"
- note removed: "Charged"
- note removed: "Charging"
- note removed: "Display"
- note removed: "Microcontroller"
- note removed: "Negative Power Supply"
- note removed: "Note: hold SW1 down when programming"
- note removed: "Peak Detector"
- note removed: "Power Switch"
- note removed: "USB Charger"
- note removed: "Voltage Reference"
- note removed: "Wien Bridge Oscillator"
